Commit message: Added URDF - Estimated values. Will retune after redesign and receive components.

File: ws_robot/src/ugv_description/urdf/physical_description/robot_base.xacro (robot description, xacro)
@@ -1,12 +1,14 @@
 <?xml version="1.0"?>
 <robot xmlns:xacro="http://www.ros.org/wiki/xacro">
-    <!-- BASE -->
+    <!-- FOOTPRINT (Projection of rear axle center on the ground)-->
     <link name="base_footprint"></link>
+    <!-- BASE LINK (Center between front and rear axle) -->
     <link name="base_link">
         <visual>
-            <origin xyz="0 0 0" rpy="${pi/2} 0 0" />
+            <origin xyz="0 0 0" rpy="0 0 0" />
             <geometry>
-                <cylinder length="0.3" radius="0.01" />
+                <box size="${wheelbase} 0.01 0.01"/>
             </geometry>
+            <material name="red" />
         </visual>
     </link>
@@ -14,5 +16,83 @@
         <parent link="base_footprint" />
         <child link="base_link" />
-        <origin xyz="0.0 0.0 0.1375" rpy="0 0 0" />
+        <origin xyz="${wheelbase / 2} 0 ${wheel_radius}" rpy="0 0 0" />
+    </joint>
+    <!-- REAR AXLE & WHEELS -->
+    <link name="rear_axle_link">
+        <visual>
+            <origin xyz="0 0 0" rpy="${pi/2} 0 0" />
+            <geometry>
+                <cylinder length="${rear_track}" radius="0.005" />
+            </geometry>
+            <material name="green" />
+        </visual>
+    </link>
+    <joint name="rear_axle_joint" type="fixed">
+        <parent link="base_link" />
+        <child link="rear_axle_link" />
+        <origin xyz="${-(wheelbase) / 2} 0 0" rpy="0 0 0" />
+    </joint>
+    <!-- BR Wheel -->
+    <xacro:wheel_link prefix="rear_right" />
+    <joint name="rear_right_wheel_joint" type="continuous">
+        <parent link="rear_axle_link" />
+        <child link="rear_right_wheel_link" />
+        <origin xyz="0 ${-(rear_track / 2)} 0" rpy="0 0 0" />
+        <axis xyz="0 1 0" />
+    </joint>
+    <!-- BL Wheel -->
+    <xacro:wheel_link prefix="rear_left" />
+    <joint name="rear_left_wheel_joint" type="continuous">
+        <parent link="rear_axle_link" />
+        <child link="rear_left_wheel_link" />
+        <origin xyz="0 ${(rear_track / 2)} 0" rpy="0 0 0" />
+        <axis xyz="0 1 0" />
+    </joint>
+    <!-- FRONT AXLE & WHEELS -->
+    <link name="front_axle_link">
+        <visual>
+            <origin xyz="0 0 0" rpy="${pi/2} 0 0" />
+            <geometry>
+                <cylinder length="${front_track}" radius="0.005" />
+            </geometry>
+            <material name="green" />
+        </visual>
+    </link>
+    <joint name="front_axle_joint" type="fixed">
+        <parent link="base_link" />
+        <child link="front_axle_link" />
+        <origin xyz="${wheelbase / 2} 0 0" rpy="0 0 0" />
+    </joint>
+    <!-- FR Wheel -->
+    <xacro:steering_link prefix="front_right" />
+    <joint name="front_right_steer_joint" type="revolute">
+        <parent link="front_axle_link" />
+        <child link="front_right_steering_link" />
+        <origin xyz="0 ${-((front_track / 2)-(wheel_width / 2))} 0" rpy="0 0 0" />
+        <axis xyz="0 0 1" />
+        <limit lower="-${max_steering_angle}" upper="${max_steering_angle}" effort="200" velocity="20" />
+    </joint>
+    <xacro:wheel_link prefix="front_right" />
+    <joint name="front_right_wheel_joint" type="continuous">
+        <parent link="front_right_steering_link" />
+        <child link="front_right_wheel_link" />
+        <origin xyz="0 ${-(wheel_width / 2)} 0" rpy="0 0 0" />
+        <axis xyz="0 1 0" />
+    </joint>
+    <!-- FL Wheel -->
+    <xacro:steering_link prefix="front_left" />
+    <joint name="front_left_steer_joint" type="revolute">
+        <parent link="front_axle_link" />
+        <child link="front_left_steering_link" />
+        <origin xyz="0 ${((front_track / 2)-(wheel_width / 2))} 0" rpy="0 0 0" />
+        <axis xyz="0 0 1" />
+        <limit lower="-${max_steering_angle}" upper="${max_steering_angle}" effort="200" velocity="20" />
+    </joint>
+    <xacro:wheel_link prefix="front_left" />
+    <joint name="front_left_wheel_joint" type="continuous">
+        <parent link="front_left_steering_link" />
+        <child link="front_left_wheel_link" />
+        <origin xyz="0 ${wheel_width / 2} 0" rpy="0 0 0" />
+        <axis xyz="0 1 0" />
     </joint>
 </robot>

File: ws_robot/src/ugv_description/urdf/physical_description/robot_hat.xacro (robot description, xacro)
@@ -1,20 +1,67 @@
 <?xml version="1.0"?>
 <robot xmlns:xacro="http://www.ros.org/wiki/xacro">
-    <!-- Hat Base -->
-    <link name="hat_link">
-        <visual name="">
-            <origin xyz="0.0 0.0 -0.16" rpy="0.0 0.0 0.0"/>
+    <!-- PLATFORM BASE -->
+    <link name="platform_link">
+        <visual>
+            <origin xyz="0 0 ${-(platform_height / 2)}" rpy="0 0 0"/>
              <geometry>
-                <mesh filename="file://$(find ugv_description)/models/hat/Hunter_SE_HAT.stl" />
+                <box size="${wheelbase} ${rear_track * 0.6} ${platform_height}"/>
             </geometry>
-            <material name="">
-                <color rgba="1.0 1.0 1.0 1.0"/>
-            </material>
+            <material name="white"/>
         </visual>
     </link>
     <joint name="hat_link_joint" type="fixed">
-        <origin xyz="-0.19 0.0 0.0" rpy="0.0 0.0 0.0"/>
         <parent link="base_link"/>
-        <child link="hat_link"/>
+        <child link="platform_link"/>
+        <origin xyz="0 0 0.05" rpy="0 0 0"/>
+    </joint>
+    <!-- LIDAR SENSOR -->
+    <!-- Hokuyo UST-10LX (Perception is at 47.4 mm from base)-->
+    <xacro:property name="ust_10lx_perception_height" value="0.0474" />
+    <link name="lidar_hky_link">
+        <visual>
+            <origin xyz="0 0 ${(0.07/2) - ust_10lx_perception_height}" rpy="0 0 0"/>
+            <geometry>
+                <cylinder radius="0.025" length="0.07"/>
+            </geometry>
+            <material name="orange"/>
+        </visual>
+    </link>
+    <joint name="lidar_hky_link_joint" type="fixed">
+        <parent link="platform_link"/>
+        <child link="lidar_hky_link"/>
+        <origin xyz="0.12 0 ${ust_10lx_perception_height + 0}" rpy="0 0 0"/>
+    </joint>
+    <!-- IMU SENSOR -->
+    <!-- VESC 6 MKVI -->
+    <link name="imu_vesc_link">
+        <visual>
+            <origin xyz="0 0 0" rpy="0 0 0"/>
+            <geometry>
+                <box size="0.07 0.075 0.017"/>
+            </geometry>
+            <material name="orange"/>
+        </visual>
+    </link>
+    <joint name="imu_vesc_link_joint" type="fixed">
+        <parent link="platform_link"/>
+        <child link="imu_vesc_link"/>
+        <origin xyz="-0.1 0 0.01428" rpy="0 0 0"/>
+    </joint>
+    <!-- CAMERA SENSOR -->
+    <!-- Logitech C920 -->
+    <link name="camera_c920_link">
+        <visual>
+            <origin xyz="0 0 0" rpy="0 0 0"/>
+            <geometry>
+                <box size="0.02412 0.09333 0.02886"/>
+            </geometry>
+            <material name="orange"/>
+        </visual>
+    </link>
+    <joint name="camera_c920_link_joint" type="fixed">
+        <parent link="platform_link"/>
+        <child link="camera_c920_link"/>
+        <origin xyz="0.08 0 0.085" rpy="0 0 0"/>
     </joint>
 </robot>

File: ws_robot/src/ugv_description/urdf/robot.urdf.xacro (robot description, xacro)
@@ -2,5 +2,8 @@
 <!-- URDF of Physical Robot -->
 <robot xmlns:xacro="http://www.ros.org/wiki/xacro"  name="ugv_hunterse">
+    <!-- Common -->
+    <xacro:include filename="physical_description/common_properties.xacro" />
     <!-- Physical Description -->
+    <xacro:include filename="physical_description/macros.xacro" />
     <xacro:include filename="physical_description/robot_base.xacro" />
     <xacro:include filename="physical_description/robot_hat.xacro" />

File: ws_robot/src/ugv_description/urdf/sim.urdf.xacro (robot description, xacro)
@@ -2,5 +2,8 @@
 <!-- URDF of Robot Simulation -->
 <robot xmlns:xacro="http://www.ros.org/wiki/xacro"  name="ugv_hunterse">
+    <!-- Common -->
+    <xacro:include filename="physical_description/common_properties.xacro" />
     <!-- Physical Description -->
+    <xacro:include filename="physical_description/macros.xacro" />
     <xacro:include filename="physical_description/robot_base.xacro" />
     <xacro:include filename="physical_description/robot_hat.xacro" />
