Commit message: Change to Hokuyo LiDAR & update URDF

File: ws_robot/src/ugv_description/urdf/physical_description/common_properties.xacro (robot description, xacro)
@@ -2,4 +2,5 @@
 <robot xmlns:xacro="http://www.ros.org/wiki/xacro">
     <!-- Traxxas Ford Fiesta ST Rally VXL -->
+    <!-- PROPERTIES -->
     <xacro:property name="wheelbase" value="0.324" />
     <xacro:property name="wheel_radius" value="0.05" />
@@ -13,5 +14,5 @@
     <xacro:property name="platform_mass" value="1.2"/>
     <xacro:property name="platform_height" value="0.005"/>
-    <!-- COLORS -->
+    <!-- VISUALIZATION COLORS -->
     <material name="white">
         <color rgba="1.0 1.0 1.0 1" />
@@ -38,31 +39,3 @@
         <color rgba="1.0 0.5 0 1" />
     </material>
-    <!-- INERTIAS -->
-    <xacro:macro name="box_inertia" params="m l w h xyz rpy">
-        <inertial>
-            <origin xyz="${xyz}" rpy="${rpy}" />
-            <mass value="${m}" />
-            <inertia ixx="${(m/12) * (h*h + l*l)}" ixy="0" ixz="0"
-                     iyy="${(m/12) * (w*w + l*l)}" iyz="0"
-                     izz="${(m/12) * (w*w + h*h)}" />
-        </inertial>
-    </xacro:macro>
-    <xacro:macro name="cylinder_inertia" params="m r h xyz rpy">
-        <inertial>
-            <origin xyz="${xyz}" rpy="${rpy}" />
-            <mass value="${m}" />
-            <inertia ixx="${(m/12) * (3*r*r + h*h)}" ixy="0" ixz="0"
-                     iyy="${(m/12) * (3*r*r + h*h)}" iyz="0"
-                     izz="${(m/2) * (r*r)}" />
-        </inertial>
-    </xacro:macro>
-    <xacro:macro name="sphere_inertia" params="m r xyz rpy">
-        <inertial>
-            <origin xyz="${xyz}" rpy="${rpy}" />
-            <mass value="${m}" />
-            <inertia ixx="${(2/5) * m * r * r}" ixy="0" ixz="0"
-                     iyy="${(2/5) * m * r * r}" iyz="0"
-                     izz="${(2/5) * m * r * r}" />
-        </inertial>
-    </xacro:macro>
 </robot>

File: ws_robot/src/ugv_description/urdf/physical_description/macros.xacro (robot description, xacro)
@@ -1,4 +1,32 @@
 <?xml version="1.0"?>
 <robot xmlns:xacro="http://www.ros.org/wiki/xacro">
+    <!-- INERTIAS -->
+    <xacro:macro name="box_inertia" params="m l w h xyz rpy">
+        <inertial>
+            <origin xyz="${xyz}" rpy="${rpy}" />
+            <mass value="${m}" />
+            <inertia ixx="${(m/12) * (h*h + l*l)}" ixy="0" ixz="0"
+                     iyy="${(m/12) * (w*w + l*l)}" iyz="0"
+                     izz="${(m/12) * (w*w + h*h)}" />
+        </inertial>
+    </xacro:macro>
+    <xacro:macro name="cylinder_inertia" params="m r h xyz rpy">
+        <inertial>
+            <origin xyz="${xyz}" rpy="${rpy}" />
+            <mass value="${m}" />
+            <inertia ixx="${(m/12) * (3*r*r + h*h)}" ixy="0" ixz="0"
+                     iyy="${(m/12) * (3*r*r + h*h)}" iyz="0"
+                     izz="${(m/2) * (r*r)}" />
+        </inertial>
+    </xacro:macro>
+    <xacro:macro name="sphere_inertia" params="m r xyz rpy">
+        <inertial>
+            <origin xyz="${xyz}" rpy="${rpy}" />
+            <mass value="${m}" />
+            <inertia ixx="${(2/5) * m * r * r}" ixy="0" ixz="0"
+                     iyy="${(2/5) * m * r * r}" iyz="0"
+                     izz="${(2/5) * m * r * r}" />
+        </inertial>
+    </xacro:macro>
     <!-- PHYSICAL DESCRIPTION MACROS -->
     <xacro:macro name="wheel_link" params="prefix">

File: ws_robot/src/ugv_description/urdf/physical_description/robot_base.xacro (robot description, xacro)
@@ -2,5 +2,5 @@
 <robot xmlns:xacro="http://www.ros.org/wiki/xacro">
     <!-- FOOTPRINT (Projection of rear axle center on the ground)-->
-    <link name="base_footprint"></link>
+    <link name="base_footprint"/>
     <!-- BASE LINK (Center between front and rear axle) -->
     <link name="base_link">

File: ws_robot/src/ugv_description/urdf/physical_description/robot_hat.xacro (robot description, xacro)
@@ -19,5 +19,5 @@
     <!-- Hokuyo UST-10LX (Perception is at 47.4 mm from base)-->
     <xacro:property name="ust_10lx_perception_height" value="0.0474" />
-    <link name="lidar_hky_link">
+    <link name="lidar_1_link">
         <visual>
             <origin xyz="0 0 ${(0.07/2) - ust_10lx_perception_height}" rpy="0 0 0"/>
@@ -28,12 +28,12 @@
         </visual>
     </link>
-    <joint name="lidar_hky_link_joint" type="fixed">
+    <joint name="lidar_1_link_joint" type="fixed">
         <parent link="platform_link"/>
-        <child link="lidar_hky_link"/>
+        <child link="lidar_1_link"/>
         <origin xyz="0.12 0 ${ust_10lx_perception_height + 0}" rpy="0 0 0"/>
     </joint>
     <!-- IMU SENSOR -->
     <!-- VESC 6 MKVI -->
-    <link name="imu_vesc_link">
+    <link name="imu_1_link">
         <visual>
             <origin xyz="0 0 0" rpy="0 0 0"/>
@@ -44,12 +44,12 @@
         </visual>
     </link>
-    <joint name="imu_vesc_link_joint" type="fixed">
+    <joint name="imu_1_link_joint" type="fixed">
         <parent link="platform_link"/>
-        <child link="imu_vesc_link"/>
+        <child link="imu_1_link"/>
         <origin xyz="-0.1 0 0.01428" rpy="0 0 0"/>
     </joint>
     <!-- CAMERA SENSOR -->
     <!-- Logitech C920 -->
-    <link name="camera_c920_link">
+    <link name="camera_1_link">
         <visual>
             <origin xyz="0 0 0" rpy="0 0 0"/>
@@ -60,8 +60,15 @@
         </visual>
     </link>
-    <joint name="camera_c920_link_joint" type="fixed">
+    <joint name="camera_1_link_joint" type="fixed">
         <parent link="platform_link"/>
-        <child link="camera_c920_link"/>
+        <child link="camera_1_link"/>
         <origin xyz="0.08 0 0.085" rpy="0 0 0"/>
     </joint>
+    <!-- REP-103 convention -->
+    <link name="camera_optical_1_link"/>
+    <joint name="camera_optical_1_link_joint" type="fixed">
+        <parent link="camera_1_link"/>
+        <child link="camera_optical_1_link"/>
+        <origin xyz="0 0 0" rpy="${-pi/2} 0 ${-pi/2}"/>
+    </joint>
 </robot>
