Commit message: Tune VESC limits, add LT speed boost and live steering joints
- VESC: brake and speed limits match the controller's own settings, now
  kept in misc/VESC (vesc_mcconf.xml, vesc_appconf.xml)
- Joystick: LT scales the teleop speed up to 5x (ugv_util/teleop_speed_multiplier)
- Model: steering and wheel joints follow the servo command and wheel
  odometry (ugv_util/vehicle_joint_state_publisher); meshes use package://
  so RViz on another computer finds them
- utility_visualizer: no crash before the first drive command
- Localization: map-frame odometry starts only when there is a map
- udev rule for the See3CAM camera

File: ws_robot/src/ugv_description/urdf/physical_description/robot_hat.xacro (robot description, xacro)
@@ -13,5 +13,5 @@
             <origin xyz="0 ${-0.145/2} -0.005" rpy="0 0 0"/>
              <geometry>
-                <mesh filename="file://$(find ugv_description)/models/platform_deck.STL"/>
+                <mesh filename="package://ugv_description/models/platform_deck.STL"/>
             </geometry>
             <material name="white"/>
@@ -20,5 +20,5 @@
             <origin xyz="0.10835 0.0485 0" rpy="${pi/2} 0 0"/>
              <geometry>
-                <mesh filename="file://$(find ugv_description)/models/platform_for_jetson_orin_nano_nx_dev_kit.STL"/>
+                <mesh filename="package://ugv_description/models/platform_for_jetson_orin_nano_nx_dev_kit.STL"/>
             </geometry>
             <material name="white"/>
@@ -27,5 +27,5 @@
             <origin xyz="0.112825 -0.036925 0.005" rpy="0 0 0"/>
              <geometry>
-                <mesh filename="file://$(find ugv_description)/models/jetson_orin_nano_dev_kit.STL"/>
+                <mesh filename="package://ugv_description/models/jetson_orin_nano_dev_kit.STL"/>
             </geometry>
             <material name="white"/>
@@ -34,5 +34,5 @@
             <origin xyz="-0.095 ${0.153/2} -0.02" rpy="${pi/2} 0 0"/>
              <geometry>
-                <mesh filename="file://$(find ugv_description)/models/rear_spoiler.STL"/>
+                <mesh filename="package://ugv_description/models/rear_spoiler.STL"/>
             </geometry>
             <material name="white"/>
@@ -58,5 +58,5 @@
             <origin xyz="${-0.025-0.008843159} ${-(0.04945/2)-0.000825} ${-ust_10lx_perception_height - 0.01}" rpy="${pi/2} 0 ${pi/2}"/>
             <geometry>
-                <mesh filename="file://$(find ugv_description)/models/hokuyo_ust_10lx_20lx.STL"/>
+                <mesh filename="package://ugv_description/models/hokuyo_ust_10lx_20lx.STL"/>
             </geometry>
             <material name="orange"/>
@@ -65,5 +65,5 @@
             <origin xyz="${-0.056/2} ${0.056/2} ${-ust_10lx_perception_height-0.01}" rpy="${pi/2} 0 0"/>
             <geometry>
-                <mesh filename="file://$(find ugv_description)/models/platform_for_ust_10lx.STL"/>
+                <mesh filename="package://ugv_description/models/platform_for_ust_10lx.STL"/>
             </geometry>
             <material name="orange"/>
@@ -88,5 +88,5 @@
             <origin xyz="${0.07/2} ${-0.015 - 0.075/2} 0" rpy="0 0 ${pi/2}"/>
             <geometry>
-                <mesh filename="file://$(find ugv_description)/models/vesc6.STL"/>
+                <mesh filename="package://ugv_description/models/vesc6.STL"/>
             </geometry>
             <material name="orange"/>
@@ -111,5 +111,5 @@
             <origin xyz="0.1 0.047 -0.02898" rpy="${pi/2} 0 ${-pi/2}"/>
             <geometry>
-                <mesh filename="file://$(find ugv_description)/models/logitech_c920_webcam.STL"/>
+                <mesh filename="package://ugv_description/models/logitech_c920_webcam.STL"/>
             </geometry>
             <material name="orange"/>
